File: LIC_rack_BB-00.brd (EAGLE design)
At the start: 162 x 102 mm, 22 parts, among them IC1 74HC125D, IC3 74HC125D, IC4 MEGA128-A, IC6 MAX481CSA, Q1 14.7456, U1 ATPROG-V

Commit message: Pridan
Pridan pouze obrazek desky pro vyrobu
Connections:
- new net N$1: J1.A22
Changed lines of the file:
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@@
 <layer number="20" name="Dimension" color="15" fill="1" visible="yes" active="yes"/>
 <layer number="21" name="tPlace" color="7" fill="1" visible="yes" active="yes"/>
-<layer number="22" name="bPlace" color="7" fill="1" visible="yes" active="yes"/>
+<layer number="22" name="bPlace" color="7" fill="1" visible="no" active="yes"/>
 <layer number="23" name="tOrigins" color="15" fill="1" visible="yes" active="yes"/>
-<layer number="24" name="bOrigins" color="15" fill="1" visible="yes" active="yes"/>
+<layer number="24" name="bOrigins" color="15" fill="1" visible="no" active="yes"/>
 <layer number="25" name="tNames" color="7" fill="1" visible="yes" active="yes"/>
-<layer number="26" name="bNames" color="7" fill="1" visible="yes" active="yes"/>
+<layer number="26" name="bNames" color="7" fill="1" visible="no" active="yes"/>
 <layer number="27" name="tValues" color="7" fill="1" visible="yes" active="yes"/>
-<layer number="28" name="bValues" color="7" fill="1" visible="yes" active="yes"/>
+<layer number="28" name="bValues" color="7" fill="1" visible="no" active="yes"/>
 <layer number="29" name="tStop" color="7" fill="3" visible="no" active="yes"/>
 <layer number="30" name="bStop" color="7" fill="6" visible="no" active="yes"/>
@@
 <layer number="50" name="dxf" color="7" fill="1" visible="no" active="yes"/>
 <layer number="51" name="tDocu" color="7" fill="1" visible="yes" active="yes"/>
-<layer number="52" name="bDocu" color="7" fill="1" visible="yes" active="yes"/>
+<layer number="52" name="bDocu" color="7" fill="1" visible="no" active="yes"/>
 <layer number="53" name="tGND_GNDA" color="7" fill="9" visible="no" active="no"/>
 <layer number="54" name="bGND_GNDA" color="1" fill="9" visible="no" active="no"/>
@@
 <layer number="97" name="Info" color="7" fill="1" visible="no" active="no"/>
 <layer number="98" name="Guide" color="6" fill="1" visible="no" active="no"/>
-<layer number="100" name="PaJa" color="12" fill="7" visible="yes" active="yes"/>
-<layer number="101" name="Doplnky" color="5" fill="1" visible="yes" active="yes"/>
-<layer number="102" name="Kola" color="11" fill="7" visible="yes" active="yes"/>
+<layer number="100" name="PaJa" color="12" fill="7" visible="no" active="yes"/>
+<layer number="101" name="Doplnky" color="5" fill="1" visible="no" active="yes"/>
+<layer number="102" name="Kola" color="11" fill="7" visible="no" active="yes"/>
 <layer number="103" name="Popisy" color="7" fill="1" visible="yes" active="yes"/>
 <layer number="104" name="Zapojeni" color="7" fill="1" visible="yes" active="yes"/>
 <layer number="105" name="tPlate" color="7" fill="1" visible="yes" active="yes"/>
-<layer number="106" name="bPlate" color="7" fill="1" visible="yes" active="yes"/>
+<layer number="106" name="bPlate" color="7" fill="1" visible="no" active="yes"/>
 <layer number="107" name="Crop" color="7" fill="1" visible="no" active="no"/>
-<layer number="110" name="wago-seda" color="7" fill="8" visible="yes" active="yes"/>
-<layer number="111" name="wago-cervena" color="12" fill="8" visible="yes" active="yes"/>
-<layer number="112" name="wago-zelena" color="2" fill="8" visible="yes" active="yes"/>
-<layer number="113" name="wago-modra" color="1" fill="8" visible="yes" active="yes"/>
+<layer number="110" name="wago-seda" color="7" fill="8" visible="no" active="yes"/>
+<layer number="111" name="wago-cervena" color="12" fill="8" visible="no" active="yes"/>
+<layer number="112" name="wago-zelena" color="2" fill="8" visible="no" active="yes"/>
+<layer number="113" name="wago-modra" color="1" fill="8" visible="no" active="yes"/>
 <layer number="116" name="centerDrill" color="7" fill="1" visible="no" active="yes"/>
 <layer number="121" name="_tsilk" color="7" fill="1" visible="no" active="no"/>
@@
 <wire x1="61.542" y1="-15.691" x2="63.951" y2="-15.691" width="0.3048" layer="1"/>
 </signal>
+<signal name="N$1">
+<contactref element="J1" pad="A22"/>
+</signal>
 </signals>
