File: LIC_rack_BB-00.sch (EAGLE design)
At the start: 22 parts, among them IC1 74HC125D, IC3 74HC125D, IC4 MEGA128-A, IC6 MAX481CSA, Q1 14.7456, U1 ATPROG-V

Commit message: Pridan
Pridan pouze obrazek desky pro vyrobu
Connections:
- new net N$1: J1-A22.MS
Changed lines of the file:
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@@
+</segment>
+</net>
+<net name="N$1" class="0">
+<segment>
+<pinref part="J1" gate="-A22" pin="MS"/>
+<wire x1="220.98" y1="104.14" x2="208.28" y2="104.14" width="0.1524" layer="91"/>
 </segment>
 </net>
