File: LIC_Rack_BB-01_ext.brd (EAGLE design)
At the start: 29.2 x 28.9 mm, 6 parts, among them Q1 IRLL014

Commit message: Upravy
Connections:
- net +5V: no longer K3.2, K3.4, K3.6
- net GND: now also K3.2, K3.4, K3.6
Routing:
- net +5V: track 55.3 -> 0.00 mm
Changed lines of the file:
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@@
 <wire x1="6.35" y1="27.94" x2="5.08" y2="26.67" width="0.6096" layer="16"/>
 <wire x1="5.08" y1="26.67" x2="5.08" y2="25.4" width="0.6096" layer="16"/>
+<contactref element="K3" pad="2"/>
+<contactref element="K3" pad="4"/>
+<contactref element="K3" pad="6"/>
+<wire x1="24.13" y1="7.62" x2="24.13" y2="12.7" width="0" layer="19" extent="1-1"/>
+<wire x1="24.13" y1="2.54" x2="24.13" y2="7.62" width="0" layer="19" extent="1-1"/>
+<wire x1="24.13" y1="21.59" x2="24.13" y2="12.7" width="0" layer="19" extent="1-1"/>
 </signal>
 <signal name="PA7">
@@
 <signal name="+5V">
 <contactref element="REL1" pad="+3"/>
-<contactref element="K3" pad="2"/>
-<contactref element="K3" pad="4"/>
-<contactref element="K3" pad="6"/>
 <contactref element="K4" pad="4"/>
-<wire x1="15.24" y1="25.4" x2="16.51" y2="25.4" width="0.6096" layer="16"/>
-<wire x1="16.51" y1="25.4" x2="17.78" y2="24.13" width="0.6096" layer="16"/>
-<wire x1="17.78" y1="24.13" x2="17.78" y2="21.59" width="0.6096" layer="16"/>
-<wire x1="17.78" y1="21.59" x2="20.32" y2="21.59" width="0.6096" layer="16"/>
-<wire x1="20.32" y1="21.59" x2="21.59" y2="20.32" width="0.6096" layer="16"/>
-<wire x1="21.59" y1="20.32" x2="21.59" y2="19.05" width="0.6096" layer="16"/>
-<wire x1="21.59" y1="19.05" x2="22.86" y2="17.78" width="0.6096" layer="16"/>
-<wire x1="22.86" y1="17.78" x2="25.4" y2="17.78" width="0.6096" layer="16"/>
-<wire x1="25.4" y1="17.78" x2="26.67" y2="16.51" width="0.6096" layer="16"/>
-<wire x1="26.67" y1="16.51" x2="26.67" y2="13.97" width="0.6096" layer="16"/>
-<wire x1="26.67" y1="13.97" x2="25.4" y2="12.7" width="0.6096" layer="16"/>
-<wire x1="24.13" y1="12.7" x2="25.4" y2="12.7" width="0.6096" layer="16"/>
-<wire x1="25.4" y1="12.7" x2="26.67" y2="11.43" width="0.6096" layer="16"/>
-<wire x1="26.67" y1="11.43" x2="26.67" y2="8.89" width="0.6096" layer="16"/>
-<wire x1="26.67" y1="8.89" x2="25.4" y2="7.62" width="0.6096" layer="16"/>
-<wire x1="25.4" y1="7.62" x2="24.13" y2="7.62" width="0.6096" layer="16"/>
-<wire x1="24.13" y1="2.54" x2="25.4" y2="2.54" width="0.6096" layer="16"/>
-<wire x1="25.4" y1="2.54" x2="26.67" y2="3.81" width="0.6096" layer="16"/>
-<wire x1="26.67" y1="3.81" x2="26.67" y2="6.35" width="0.6096" layer="16"/>
-<wire x1="26.67" y1="6.35" x2="25.4" y2="7.62" width="0.6096" layer="16"/>
-<wire x1="7.62" y1="10.16" x2="19.05" y2="10.16" width="0.6096" layer="16"/>
-<wire x1="19.05" y1="10.16" x2="21.59" y2="12.7" width="0.6096" layer="16"/>
-<wire x1="21.59" y1="12.7" x2="24.13" y2="12.7" width="0.6096" layer="16"/>
+<wire x1="7.62" y1="10.16" x2="15.24" y2="25.4" width="0" layer="19" extent="1-1"/>
 </signal>
 <signal name="IN_LASER">
