File: LIC_rack_BB-01.sch (EAGLE design)
At the start: 22 parts, among them IC1 74HC125D, IC3 74HC125D, IC4 MEGA128-A, IC6 MAX481CSA, Q1 14.7456, U1 ATPROG-V

Commit message: Upravy
Parts:
- added JUM8, JUM9: S1G3_JUMP, #PaJa_konektory:S1G3_JUMP
Connections:
- net N$1 renamed PA7-LASER
- new net N$3: JUM8.1
- new net N$4: JUM8.3
- new net N$6: JUM9.1
- new net N$7: JUM9.3
- new net PE0: JUM9.2
- new net PE1: JUM8.2
- net +5V: now also R1.1, R3.1, R4.1
- net GND: no longer R1.1, R3.1, R4.1
Other:
- moved on the sheet: R1, R3, R4
Changed lines of the file:
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@@
 <part name="JUM5" library="#PaJa_konektory" deviceset="S1G2_JUMP" device=""/>
 <part name="R4" library="#PaJa_31" deviceset="R" device="_1206" value="10k"/>
+<part name="JUM8" library="#PaJa_konektory" deviceset="S1G3_JUMP" device=""/>
+<part name="JUM9" library="#PaJa_konektory" deviceset="S1G3_JUMP" device=""/>
 </parts>
 <sheets>
@@
 <instance part="P+3" gate="1" x="55.88" y="160.02"/>
 <instance part="GND3" gate="1" x="50.8" y="68.58"/>
-<instance part="R1" gate="R" x="157.48" y="60.96" rot="R90"/>
-<instance part="R3" gate="R" x="200.66" y="60.96" rot="R90"/>
-<instance part="R4" gate="R" x="238.76" y="60.96" rot="R90"/>
+<instance part="R1" gate="R" x="157.48" y="86.36" rot="R270"/>
+<instance part="R3" gate="R" x="200.66" y="86.36" rot="R270"/>
+<instance part="R4" gate="R" x="238.76" y="86.36" rot="R270"/>
+<instance part="JUM8" gate="JUMP" x="180.34" y="149.86"/>
+<instance part="JUM9" gate="JUMP" x="215.9" y="132.08"/>
 </instances>
 <busses>
@@
 <junction x="50.8" y="83.82"/>
 </segment>
-<segment>
-<pinref part="R1" gate="R" pin="1"/>
-<wire x1="157.48" y1="55.88" x2="157.48" y2="50.8" width="0.1524" layer="91"/>
-<label x="157.48" y="50.8" size="1.016" layer="95" xref="yes"/>
-</segment>
-<segment>
-<pinref part="R3" gate="R" pin="1"/>
-<wire x1="200.66" y1="55.88" x2="200.66" y2="50.8" width="0.1524" layer="91"/>
-<label x="200.66" y="50.8" size="1.016" layer="95" xref="yes"/>
-</segment>
-<segment>
-<pinref part="R4" gate="R" pin="1"/>
-<wire x1="238.76" y1="55.88" x2="238.76" y2="50.8" width="0.1524" layer="91"/>
-<label x="238.76" y="50.8" size="1.016" layer="95" xref="yes"/>
-</segment>
 </net>
 <net name="+5V" class="0">
@@
 <junction x="55.88" y="152.4"/>
 </segment>
+<segment>
+<pinref part="R3" gate="R" pin="1"/>
+<wire x1="200.66" y1="91.44" x2="208.28" y2="91.44" width="0.1524" layer="91"/>
+<label x="208.28" y="91.44" size="1.016" layer="95" xref="yes"/>
+</segment>
+<segment>
+<pinref part="R1" gate="R" pin="1"/>
+<wire x1="157.48" y1="91.44" x2="167.64" y2="91.44" width="0.1524" layer="91"/>
+<label x="167.64" y="91.44" size="1.016" layer="95" xref="yes"/>
+</segment>
+<segment>
+<pinref part="R4" gate="R" pin="1"/>
+<wire x1="238.76" y1="91.44" x2="243.84" y2="91.44" width="0.1524" layer="91"/>
+<label x="243.84" y="91.44" size="1.016" layer="95" xref="yes"/>
+</segment>
 </net>
 <net name="P1_!RST" class="0">
@@
 <segment>
 <pinref part="R3" gate="R" pin="2"/>
-<wire x1="200.66" y1="66.04" x2="200.66" y2="71.12" width="0.1524" layer="91"/>
+<wire x1="200.66" y1="81.28" x2="200.66" y2="71.12" width="0.1524" layer="91"/>
 <wire x1="200.66" y1="71.12" x2="190.5" y2="71.12" width="0.1524" layer="91"/>
-<wire x1="200.66" y1="71.12" x2="200.66" y2="76.2" width="0.1524" layer="91"/>
-<wire x1="200.66" y1="76.2" x2="208.28" y2="76.2" width="0.1524" layer="91"/>
+<wire x1="200.66" y1="71.12" x2="200.66" y2="68.58" width="0.1524" layer="91"/>
+<wire x1="200.66" y1="68.58" x2="208.28" y2="68.58" width="0.1524" layer="91"/>
 <label x="190.5" y="71.12" size="1.016" layer="95" rot="R180" xref="yes"/>
 <junction x="200.66" y="71.12"/>
@@
 <segment>
 <wire x1="149.86" y1="71.12" x2="157.48" y2="71.12" width="0.1524" layer="91"/>
-<wire x1="157.48" y1="71.12" x2="157.48" y2="76.2" width="0.1524" layer="91"/>
-<wire x1="157.48" y1="76.2" x2="165.1" y2="76.2" width="0.1524" layer="91"/>
-<wire x1="157.48" y1="71.12" x2="157.48" y2="66.04" width="0.1524" layer="91"/>
+<wire x1="157.48" y1="71.12" x2="157.48" y2="68.58" width="0.1524" layer="91"/>
+<wire x1="157.48" y1="68.58" x2="165.1" y2="68.58" width="0.1524" layer="91"/>
+<wire x1="157.48" y1="71.12" x2="157.48" y2="81.28" width="0.1524" layer="91"/>
 <pinref part="R1" gate="R" pin="2"/>
 <label x="149.86" y="71.12" size="1.016" layer="95" rot="R180" xref="yes"/>
@@
 <segment>
 <pinref part="R4" gate="R" pin="2"/>
-<wire x1="238.76" y1="66.04" x2="238.76" y2="71.12" width="0.1524" layer="91"/>
+<wire x1="238.76" y1="81.28" x2="238.76" y2="71.12" width="0.1524" layer="91"/>
 <wire x1="238.76" y1="71.12" x2="228.6" y2="71.12" width="0.1524" layer="91"/>
-<wire x1="238.76" y1="71.12" x2="238.76" y2="76.2" width="0.1524" layer="91"/>
-<wire x1="238.76" y1="76.2" x2="246.38" y2="76.2" width="0.1524" layer="91"/>
+<wire x1="238.76" y1="71.12" x2="238.76" y2="68.58" width="0.1524" layer="91"/>
+<wire x1="238.76" y1="68.58" x2="246.38" y2="68.58" width="0.1524" layer="91"/>
 <label x="228.6" y="71.12" size="1.016" layer="95" rot="R180" xref="yes"/>
 <junction x="238.76" y="71.12"/>
@@
 <wire x1="114.3" y1="40.64" x2="121.92" y2="40.64" width="0.1524" layer="91"/>
 <label x="121.92" y="40.64" size="1.016" layer="95" xref="yes"/>
+</segment>
+</net>
+<net name="N$3" class="0">
+<segment>
+<pinref part="JUM8" gate="JUMP" pin="1"/>
+<wire x1="177.8" y1="147.32" x2="177.8" y2="139.7" width="0.1524" layer="91"/>
+<wire x1="177.8" y1="139.7" x2="170.18" y2="139.7" width="0.1524" layer="91"/>
+<label x="170.18" y="139.7" size="1.27" layer="95" ratio="12" rot="R180" xref="yes"/>
+</segment>
+</net>
+<net name="N$4" class="0">
+<segment>
+<pinref part="JUM8" gate="JUMP" pin="3"/>
+<wire x1="182.88" y1="147.32" x2="182.88" y2="139.7" width="0.1524" layer="91"/>
+<wire x1="182.88" y1="139.7" x2="190.5" y2="139.7" width="0.1524" layer="91"/>
+<label x="190.5" y="139.7" size="1.27" layer="95" ratio="12" xref="yes"/>
+</segment>
+</net>
+<net name="N$6" class="0">
+<segment>
+<pinref part="JUM9" gate="JUMP" pin="1"/>
+<wire x1="213.36" y1="129.54" x2="213.36" y2="121.92" width="0.1524" layer="91"/>
+<wire x1="213.36" y1="121.92" x2="205.74" y2="121.92" width="0.1524" layer="91"/>
+<label x="205.74" y="121.92" size="1.27" layer="95" ratio="12" rot="R180" xref="yes"/>
+</segment>
+</net>
+<net name="N$7" class="0">
+<segment>
+<pinref part="JUM9" gate="JUMP" pin="3"/>
+<wire x1="218.44" y1="129.54" x2="218.44" y2="121.92" width="0.1524" layer="91"/>
+<wire x1="218.44" y1="121.92" x2="228.6" y2="121.92" width="0.1524" layer="91"/>
+<label x="228.6" y="121.92" size="1.27" layer="95" ratio="12" xref="yes"/>
+</segment>
+</net>
+<net name="PE1" class="0">
+<segment>
+<pinref part="JUM8" gate="JUMP" pin="2"/>
+<wire x1="180.34" y1="147.32" x2="180.34" y2="134.62" width="0.1524" layer="91"/>
+<wire x1="180.34" y1="134.62" x2="170.18" y2="134.62" width="0.1524" layer="91"/>
+<label x="170.18" y="134.62" size="1.27" layer="95" ratio="12" rot="R180" xref="yes"/>
+</segment>
+</net>
+<net name="PE0" class="0">
+<segment>
+<pinref part="JUM9" gate="JUMP" pin="2"/>
+<wire x1="215.9" y1="129.54" x2="215.9" y2="116.84" width="0.1524" layer="91"/>
+<wire x1="215.9" y1="116.84" x2="205.74" y2="116.84" width="0.1524" layer="91"/>
+<label x="205.74" y="116.84" size="1.27" layer="95" ratio="12" rot="R180" xref="yes"/>
 </segment>
 </net>
@@
 <text x="238.76" y="114.3" size="1.778" layer="97" font="vector">Channel 1-4
 Output</text>
-<text x="236.474" y="98.298" size="1.778" layer="97" font="vector">Interrupt 4-5
+<text x="236.474" y="93.218" size="1.778" layer="97" font="vector">Interrupt 4-5
 InterLock</text>
 <wire x1="228.6" y1="85.09" x2="254" y2="85.09" width="0.4064" layer="97" style="longdash"/>
@@
 </segment>
 </net>
-<net name="N$1" class="0">
+<net name="PA7-LASER" class="0">
 <segment>
 <pinref part="J1" gate="-A22" pin="MS"/>
 <wire x1="220.98" y1="104.14" x2="208.28" y2="104.14" width="0.1524" layer="91"/>
-</segment>
-</net>
+<label x="208.28" y="104.14" size="1.27" layer="95" ratio="12" rot="R180" xref="yes"/>
+</segment>
+</net>
